File: ai03tutorial.sch (KiCad schematic (older format))
At the start: 24 parts

Commit message: finished electrical design phase2
Parts:
- C1: renamed from C; footprint (none) -> Capacitor_SMD:C_0805_2012Metric
- C2, C3, C4, C5, C6, C7: renamed from C?; footprint (none) -> Capacitor_SMD:C_0805_2012Metric
- D.0.0, D.0.1, D.1.0, D.1.1: renamed from D?; footprint (none) -> Diode_SMD:D_SOD-123
- F1: renamed from F?; footprint (none) -> Fuse:Fuse_1206_3216Metric
- MX.0.0, MX.0.1, MX.1.0, MX.1.1: renamed from MX?; footprint (none) -> kbd:CherryMX_1u
- R1, R2, R4: renamed from R; footprint (none) -> Resistor_SMD:R_0805_2012Metric
- R3: renamed from R?; footprint (none) -> Resistor_SMD:R_0805_2012Metric
- SW1: renamed from SW?; footprint (none) -> random-keyboard-parts:SKQG-1155865
- USB1: renamed from USB?; footprint (none) -> random-keyboard-parts:Molex-0548190589
- Y1: renamed from Y?; footprint (none) -> Crystal:Crystal_SMD_3225-4Pin_3.2x2.5mm
- renumbered U to U1
